File: sch/DCC cDecoder.brd (EAGLE design)
At the start: 285 x 10 mm, 80 parts, among them IC1 L78L05ACUTR, T1 SI9945BDY, U1 ATTINY85-20S

Commit message: version 2
Parts:
- removed VCC: (no value), wirepad:SMD1,27-2,54
- added AUX1.1: AUX1.1, wirepad:SMD1,27-2,54
- added VCC3: VCC3, wirepad:SMD1,27-2,54
- AC1.1: value (none) -> AC1.1
- AC1.2: value (none) -> AC1.2
- AC1.3: value (none) -> AC1.3
- AC2.1: value (none) -> AC2.1
- AC2.2: value (none) -> AC2.2
- AC2.3: value (none) -> AC2.3
- AUX1.2: value (none) -> AUX1.2
- AUX2.1: value (none) -> AUX2.1
- AUX2.2: value (none) -> AUX2.2
- R10, R2, R3, R4, R5, R6, R7, R8, R9: value 4.7 -> 4.7k
- SJ17, SJ18, SJ19, SJ20, SJ21, SJ22, SJ23, SJ24: device _smd:SJC -> jumper:SJ
- VCC1: value (none) -> VCC1
- VCC2: value (none) -> VCC2
- moved VCC1 281.1 mm to (283.0, 2.00)
- moved R1 2.08 mm to (18.0, 5.08)
- moved R3 2.04 mm to (74.1, 5.03)
- moved R4 2.04 mm to (102.2, 5.03)
- moved R6 1.92 mm to (158.4, 4.91)
- moved R5 1.91 mm to (130.4, 4.91)
- moved R8 1.91 mm to (214.7, 4.91)
- moved R9 1.91 mm to (242.9, 4.91)
- moved R10 1.91 mm to (273.0, 4.91)
- moved R2 1.91 mm to (46.1, 4.91)
- moved R7 1.91 mm to (186.8, 4.91)
- moved SJ18 0.21 mm to (85.3, 5.21)
- moved SJ21 0.09 mm to (169.6, 5.08)
- moved SJ17 0.09 mm to (57.1, 5.08)
- moved SJ24 0.09 mm to (254.1, 5.08)
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- renumbered + to AC1.2, +1 to AC1.1, +2 to AC1.3, - to AC2.1, -1 to AC2.2, -2 to AC2.3, AUX1 to AUX1.2, AUX2 to AUX2.2, VCC.2 to VCC2
Connections:
- removed net N$55: AUX1.2.1, LED10.C, SJ24.2
- new net N$34: AUX1.1.1, AUX1.2.1, LED10.C, SJ24.2
- net N$31: now also VCC1.1; no longer VCC.1
- net VCC: now also VCC3.1; no longer VCC1.1
Routing:
- net N$34: track 0.18 -> 32.0 mm, vias 0 -> 1
- net N$55: track 29.0 -> 0.00 mm
- net RAIL2: track 57.6 -> 82.2 mm, vias 2 -> 1
- net GND: track 66.2 -> 57.7 mm
- net VCC: track 60.6 -> 68.0 mm, vias 3 -> 2
- net +5V: track 13.8 -> 8.89 mm
- net N$65: track 3.81 -> 0.00 mm
- net N$48: track 49.0 -> 45.4 mm, vias 3 -> 2
- net N$45: track 0.00 -> 2.48 mm
- net N$36: track 0.18 -> 2.54 mm
- net AUX2: track 18.7 -> 16.5 mm
- net N$12: track 26.7 -> 28.7 mm
- net N$3: track 26.7 -> 28.7 mm
- net N$9: track 26.7 -> 28.7 mm
- net N$7: track 26.7 -> 28.6 mm
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Other:
- board text added: "AUX1"
- board text removed: "Rail"
