File: sch/DCC cDecoder.brd (EAGLE design)
At the start: 285 x 10 mm, 81 parts, among them IC1 L78L05ACUTR, T1 SI9945BDY, U1 ATTINY85-20S

Commit message: footprint mosfet changed (v3)
Parts:
- T1: device zetex:SM8 -> zetex:SO8
Routing:
- net N$48: track 45.4 -> 47.3 mm
- net N$15: track 50.1 -> 51.5 mm
- net GND: track 57.7 -> 58.9 mm
- net AUX2: track 16.5 -> 17.0 mm
Other:
- board text added: "cDecoder 26.11.2022 AZ v3"
- board text removed: "cDecoder 26.11.2022 AZ v2"
Changed lines of the file:
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@@
 <wire x1="44.577" y1="4.318" x2="44.577" y2="5.461" width="0.254" layer="25"/>
 <wire x1="44.196" y1="4.318" x2="44.958" y2="4.318" width="0.254" layer="25"/>
-<text x="6.35" y="0.381" size="0.6096" layer="21">cDecoder 26.11.2022 AZ v2</text>
+<text x="6.35" y="0.381" size="0.6096" layer="21">cDecoder 26.11.2022 AZ v3</text>
 <text x="3.302" y="1.143" size="0.4064" layer="25">AC</text>
 <text x="3.556" y="7.874" size="0.4064" layer="25">AC</text>
@@
 <attribute name="VALUE" x="39.116" y="9.2018" size="1.4224" layer="27" ratio="9" rot="R180"/>
 </element>
-<element name="T1" library="zetex" library_urn="urn:adsk.eagle:library:418" package="SM8" package3d_urn="urn:adsk.eagle:package:30984/2" value="SI9945BDY" x="50.927" y="5.033" smashed="yes" rot="R180">
+<element name="T1" library="zetex" library_urn="urn:adsk.eagle:library:418" package="SO8" package3d_urn="urn:adsk.eagle:package:30987/2" value="SI9945BDY" x="50.927" y="5.033" smashed="yes" rot="R180">
 <attribute name="MF" value="" x="50.927" y="5.033" size="1.778" layer="27" rot="R180" display="off"/>
 <attribute name="MPN" value="" x="50.927" y="5.033" size="1.778" layer="27" rot="R180" display="off"/>
@@
 <attribute name="OC_FARNELL" value="unknown" x="50.927" y="5.033" size="1.778" layer="27" rot="R180" display="off"/>
 <attribute name="OC_NEWARK" value="unknown" x="50.927" y="5.033" size="1.778" layer="27" rot="R180" display="off"/>
-<attribute name="POPULARITY" value="0" x="50.927" y="5.033" size="1.778" layer="27" rot="R180" display="off"/>
+<attribute name="POPULARITY" value="1" x="50.927" y="5.033" size="1.778" layer="27" rot="R180" display="off"/>
 <attribute name="VALUE" x="54.3062" y="8.123" size="1.27" layer="27" rot="R270"/>
 </element>
@@
 <wire x1="53.1876" y1="7.3152" x2="51.6636" y2="5.7912" width="0.1524" layer="1"/>
 <wire x1="53.1876" y1="8.0772" x2="53.1876" y2="7.3152" width="0.1524" layer="1"/>
-<wire x1="50.292" y1="8.0772" x2="50.165" y2="8.1318" width="0.1524" layer="1"/>
-<wire x1="53.1876" y1="8.0772" x2="53.213" y2="8.1318" width="0.1524" layer="1"/>
+<wire x1="50.292" y1="8.0772" x2="50.292" y2="7.633" width="0.1524" layer="1"/>
+<wire x1="53.1876" y1="8.0772" x2="52.832" y2="7.633" width="0.1524" layer="1"/>
 <wire x1="42.3672" y1="6.858" x2="39.9288" y2="6.858" width="0.1524" layer="1"/>
 <wire x1="42.672" y1="7.1628" x2="42.3672" y2="6.858" width="0.1524" layer="1"/>
@@
 <wire x1="39.7764" y1="6.7056" x2="39.906" y2="6.811" width="0.1524" layer="1"/>
 <wire x1="56.4255" y1="8" x2="53.3448" y2="8" width="0.1524" layer="1"/>
-<wire x1="53.3448" y1="8" x2="53.213" y2="8.1318" width="0.1524" layer="1"/>
+<wire x1="53.3448" y1="8" x2="52.832" y2="7.633" width="0.1524" layer="1"/>
 </signal>
 <signal name="N$33">
@@
 <wire x1="34.8996" y1="5.6388" x2="37.338" y2="8.0772" width="0.1524" layer="1"/>
 <wire x1="33.3756" y1="5.6388" x2="34.8996" y2="5.6388" width="0.1524" layer="1"/>
-<wire x1="48.6156" y1="8.0772" x2="48.641" y2="8.1318" width="0.1524" layer="1"/>
+<wire x1="48.6156" y1="8.0772" x2="49.022" y2="7.633" width="0.1524" layer="1"/>
 <wire x1="33.3756" y1="5.6388" x2="33.246" y2="5.541" width="0.1524" layer="1"/>
 </signal>
@@
 <wire x1="35.052" y1="6.7056" x2="42.2148" y2="6.7056" width="0.1524" layer="16"/>
 <wire x1="33.3756" y1="6.7056" x2="35.052" y2="6.7056" width="0.1524" layer="1"/>
-<wire x1="51.6636" y1="8.0772" x2="51.689" y2="8.1318" width="0.1524" layer="1"/>
+<wire x1="51.6636" y1="8.0772" x2="51.562" y2="7.633" width="0.1524" layer="1"/>
 <wire x1="33.3756" y1="6.7056" x2="33.246" y2="6.811" width="0.1524" layer="1"/>
 <via x="51.3588" y="6.4008" extent="1-16" drill="0.35"/>
@@
 <wire x1="1.905" y1="6.096" x2="2.01" y2="6.096" width="0.1524" layer="16"/>
 <wire x1="50.1396" y1="1.9812" x2="48.768" y2="1.9812" width="0.1524" layer="1"/>
-<wire x1="48.768" y1="1.9812" x2="48.641" y2="1.9342" width="0.1524" layer="1"/>
-<wire x1="50.1396" y1="1.9812" x2="50.165" y2="1.9342" width="0.1524" layer="1"/>
+<wire x1="48.768" y1="1.9812" x2="49.022" y2="2.433" width="0.1524" layer="1"/>
+<wire x1="50.1396" y1="1.9812" x2="50.292" y2="2.433" width="0.1524" layer="1"/>
 <wire x1="15.6972" y1="6.096" x2="2.01" y2="6.096" width="0.1524" layer="16"/>
 <wire x1="18.7452" y1="3.048" x2="15.6972" y2="6.096" width="0.1524" layer="16"/>
 <wire x1="47.5488" y1="3.048" x2="18.7452" y2="3.048" width="0.1524" layer="16"/>
 <wire x1="48.6156" y1="1.9812" x2="47.5488" y2="3.048" width="0.1524" layer="1"/>
-<wire x1="48.6156" y1="1.9812" x2="48.641" y2="1.9342" width="0.1524" layer="1"/>
+<wire x1="48.6156" y1="1.9812" x2="49.022" y2="2.433" width="0.1524" layer="1"/>
 <via x="2.01" y="6.096" extent="1-16" drill="0.35"/>
 <via x="47.5488" y="3.048" extent="1-16" drill="0.35"/>
@@
 <wire x1="53.34" y1="1.9812" x2="56.388" y2="5.0292" width="0.1524" layer="1"/>
 <wire x1="56.388" y1="5.0292" x2="56.388" y2="5.08" width="0.1524" layer="1"/>
-<wire x1="53.34" y1="1.9812" x2="53.213" y2="1.9342" width="0.1524" layer="1"/>
+<wire x1="53.34" y1="1.9812" x2="52.832" y2="2.433" width="0.1524" layer="1"/>
 <wire x1="44.5008" y1="6.096" x2="43.1292" y2="6.096" width="0.1524" layer="1"/>
 <wire x1="45.2628" y1="6.858" x2="44.5008" y2="6.096" width="0.1524" layer="1"/>
@@
 <wire x1="51.6636" y1="1.9812" x2="51.6636" y2="2.4384" width="0.1524" layer="1"/>
 <wire x1="43.1292" y1="6.096" x2="43.125" y2="6.05" width="0.1524" layer="1"/>
-<wire x1="51.6636" y1="1.9812" x2="51.689" y2="1.9342" width="0.1524" layer="1"/>
+<wire x1="51.6636" y1="1.9812" x2="51.562" y2="2.433" width="0.1524" layer="1"/>
 <wire x1="16.6116" y1="6.096" x2="15.0876" y2="6.096" width="0.1524" layer="1"/>
 <wire x1="41.91" y1="6.096" x2="16.6116" y2="6.096" width="0.1524" layer="16"/>
@@
 <wire x1="42.9768" y1="6.096" x2="43.125" y2="6.05" width="0.1524" layer="1"/>
 <wire x1="51.816" y1="1.9812" x2="53.1876" y2="1.9812" width="0.1524" layer="1"/>
-<wire x1="53.1876" y1="1.9812" x2="53.213" y2="1.9342" width="0.1524" layer="1"/>
-<wire x1="51.816" y1="1.9812" x2="51.689" y2="1.9342" width="0.1524" layer="1"/>
+<wire x1="53.1876" y1="1.9812" x2="52.832" y2="2.433" width="0.1524" layer="1"/>
+<wire x1="51.816" y1="1.9812" x2="51.562" y2="2.433" width="0.1524" layer="1"/>
 <via x="16.6116" y="6.096" extent="1-16" drill="0.35"/>
 <via x="41.91" y="6.096" extent="1-16" drill="0.35"/>
