File: sch/DCC cDecoder.sch (EAGLE design)
At the start: 80 parts, among them IC1 L78L05ACUTR, T1 SI9945BDY, U1 ATTINY85-20S

Commit message: version 2
Parts:
- removed AUX2, VCC: (no value), wirepad:SMD2
- added AUX1.2: AUX1.2, wirepad:SMD2
- added AUX2.2: AUX2.2, wirepad:SMD2
- added VCC3: VCC3, wirepad:SMD2
- AC1.1: value (none) -> AC1.1
- AC1.2: value (none) -> AC1.2
- AC1.3: value (none) -> AC1.3
- AC2.1: value (none) -> AC2.1
- AC2.2: value (none) -> AC2.2
- AC2.3: value (none) -> AC2.3
- AUX1.1: value (none) -> AUX1.1
- AUX2.1: value (none) -> AUX2.1
- R10, R2, R3, R4, R5, R6, R7, R8, R9: value 4.7 -> 4.7k
- SJ17, SJ18, SJ19, SJ20, SJ21, SJ22, SJ23, SJ24: device _smd:SJC -> jumper:SJ
- VCC1: value (none) -> VCC1
- VCC2: value (none) -> VCC2
- renumbered + to AC1.2, +1 to AC1.1, +2 to AC1.3, - to AC2.1, -1 to AC2.2, -2 to AC2.3, AUX1 to AUX1.1, VCC.2 to VCC2
Connections:
- removed net N$55: AUX1.1.P, LED10.C, SJ24.2
- new net N$34: AUX1.1.P, AUX1.2.P, LED10.C, SJ24.2
- net N$15: now also AUX2.2.P; no longer AUX2.P
- net N$31: now also VCC1.P; no longer VCC.P
- net VCC: now also VCC3.P; no longer VCC1.P
Other:
- note added: "AC"
- moved on the sheet: GND, LED1, LED10, LED2, LED3, LED4, LED5, LED6, LED7, LED8, LED9, R1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

Commit message: footprint mosfet changed (v3)
Parts:
- T1: device zetex:NMOS2SM8 -> zetex:NMOS2SO8
Changed lines of the file:
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@@
 <part name="FRAME1" library="frames" library_urn="urn:adsk.eagle:library:229" deviceset="DINA3_L" device=""/>
 <part name="U1" library="attiny25_45_85" deviceset="ATTINY85*" device="S" technology="-20"/>
-<part name="T1" library="zetex" library_urn="urn:adsk.eagle:library:418" deviceset="NMOS2SM8" device="" package3d_urn="urn:adsk.eagle:package:30984/2" value="SI9945BDY"/>
+<part name="T1" library="zetex" library_urn="urn:adsk.eagle:library:418" deviceset="NMOS2" device="SO8" package3d_urn="urn:adsk.eagle:package:30987/2" value="SI9945BDY"/>
 <part name="R11" library="rcl" library_urn="urn:adsk.eagle:library:334" deviceset="R-EU_" device="R0805" package3d_urn="urn:adsk.eagle:package:23553/2" value="22k"/>
 <part name="GND1" library="supply1" library_urn="urn:adsk.eagle:library:371" deviceset="GND" device=""/>
